File: thumb-unit-right/thumb-unit-right.kicad_pcb (KiCad board)
At the start: 2 copper layers, 82.5 x 79 mm, 24 parts, among them J1 Conn_01x10, SW1 SW_SPDT, SW2 SW_Push, SW3 SW_Push, SW4 SW_Push, SW5 SW_Push, U1 xiao-ble, U2 PMW3610, U3 TLV70218_SOT23-5

Commit message: feat: jlcpcbに発注
Parts:
- moved D2 7.86 mm to (143.4, 130.9), turned to 110 degrees
- moved J1 2.65 mm to (120.5, 133.0), turned to -90 degrees
- moved BT1 2.14 mm to (146.0, 125.0), turned to 110 degrees
- turned SW3 to -160 degrees
Routing:
- net /COL4: track 40.2 -> 65.7 mm, vias 1 -> 0
- net /ROW3: track 122.3 -> 143.7 mm, vias 2 -> 3
- net /COL2: track 95.4 -> 116.8 mm, vias 3 -> 1
- net GND: track 54.0 -> 73.8 mm, vias 9 -> 5
- net /COL1: track 78.5 -> 95.5 mm, vias 5 -> 0
- net +3V3: track 108.5 -> 94.6 mm, vias 2 -> 0
- net /MOTION: track 54.7 -> 41.8 mm, vias 1 -> 0
- net /SCLK: track 47.0 -> 36.0 mm, vias 0 -> 1
- net /COL0: track 62.3 -> 71.4 mm
- net /COL3: track 159.9 -> 168.2 mm, vias 3 -> 0
- net Net-(BT1-+): track 17.1 -> 9.70 mm
- net /BAT_SW: track 70.3 -> 77.1 mm, vias 2 -> 0
- net /ROW2: track 50.4 -> 49.4 mm, vias 0 -> 1
- net /ROW0: track 57.6 -> 56.7 mm, vias 0 -> 1
- net /SDIO: track 36.0 -> 36.9 mm, vias 0 -> 1
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